Commit message: Adds fancy urdf model of WAM-V and Velodyne PUCK

File: usv16_simulator/urdf/niceWAMV.urdf.xacro (robot description, xacro)
@@ -1,16 +1,5 @@
 <?xml version="1.0"?>
 <robot xmlns:xacro="http://www.ros.org/wiki/xacro" name="Ship">
-  <link name="Ship">
-    <inertial>
-      <origin xyz="1.51206787019308 1.78454626473221 0.280594889113911" rpy="0 0 0" />
-      <mass value="0.343059128131347" />
-      <inertia
-        ixx="1.02541857941861E-31"
-        ixy="-1.23259516440783E-32"
-        ixz="-1.7250223049292E-16"
-        iyy="0.347516126809007"
-        iyz="3.01060216944785E-47"
-        izz="0.347516126809007" />
-    </inertial>
+<link name="Ship">
     <visual>
       <origin xyz="0 0 0" rpy="0 0 0" />
@@ -22,23 +11,6 @@
       </material>
     </visual>
-    <collision>
-      <origin xyz="0 0 0" rpy="0 0 0" />
-      <geometry>
-        <mesh filename="package://usv16/meshes/Ship.STL" />
-      </geometry>
-    </collision>
   </link>
   <link name="port_pontoon">
-    <inertial>
-      <origin xyz="2.7149E-05 0.025063 0.96995" rpy="0 0 0" />
-      <mass value="862.28" />
-      <inertia
-        ixx="919.07"
-        ixy="9.5403E-05"
-        ixz="-0.018323"
-        iyy="917.35"
-        iyz="-12.94"
-        izz="1.7236" />
-    </inertial>
     <visual>
       <origin xyz="0 0 0" rpy="0 0 0" />
@@ -46,14 +18,9 @@
         <mesh filename="package://usv16/meshes/port_pontoon.STL" />
       </geometry>
-      <material name="">
+      <material
+        name="">
         <color rgba="0.50196 0.50196 0.50196 1" />
       </material>
     </visual>
-    <collision>
-      <origin xyz="0 0 0" rpy="0 0 0" />
-      <geometry>
-        <mesh filename="package://usv16/meshes/port_pontoon.STL" />
-      </geometry>
-    </collision>
   </link>
   <joint name="port_pontoon_link" type="fixed">
@@ -64,15 +31,4 @@
   </joint>
   <link name="starboard_pontoon">
-    <inertial>
-      <origin xyz="2.7148E-05 0.025067 0.96992" rpy="0 0 0" />
-      <mass value="862.3" />
-      <inertia
-        ixx="919.13"
-        ixy="9.55E-05"
-        ixz="-0.018324"
-        iyy="917.4"
-        iyz="-12.934"
-        izz="1.7242" />
-    </inertial>
     <visual>
       <origin xyz="0 0 0" rpy="0 0 0" />
@@ -84,10 +40,4 @@
       </material>
     </visual>
-    <collision>
-      <origin xyz="0 0 0" rpy="0 0 0" />
-      <geometry>
-        <mesh filename="package://usv16/meshes/starboard_pontoon.STL" />
-      </geometry>
-    </collision>
   </link>
   <joint name="starboard_pontoon_link" type="fixed">
@@ -98,16 +48,5 @@
   </joint>
   <link name="front_arm">
-    <inertial>
-      <origin xyz="1.035 0.1647 -0.056607" rpy="0 0 0" />
-      <mass value="11.056" />
-      <inertia
-        ixx="0.69846"
-        ixy="0.0042605"
-        ixz="-0.0041643"
-        iyy="3.2431"
-        iyz="-0.32611"
-        izz="3.4715" />
-    </inertial>
-    <visual>
+     <visual>
       <origin xyz="0 0 0" rpy="0 0 0" />
       <geometry>
@@ -118,10 +57,4 @@
       </material>
     </visual>
-    <collision>
-      <origin xyz="0 0 0" rpy="0 0 0" />
-      <geometry>
-        <mesh filename="package://usv16/meshes/front_arm.STL" />
-      </geometry>
-    </collision>
   </link>
   <joint name="front_arm_link" type="fixed">
@@ -132,15 +65,4 @@
   </joint>
   <link name="back_arm">
-    <inertial>
-      <origin xyz="1.0523 0.53236 -0.046184" rpy="0 0 0" />
-      <mass value="13.904" />
-      <inertia
-        ixx="0.082566"
-        ixy="-0.00023707"
-        ixz="-0.0019543"
-        iyy="0.090768"
-        iyz="-0.0085546"
-        izz="0.017971" />
-    </inertial>
     <visual>
       <origin xyz="0 0 0" rpy="0 0 0" />
@@ -152,14 +74,6 @@
       </material>
     </visual>
-    <collision>
-      <origin xyz="0 0 0" rpy="0 0 0" />
-      <geometry>
-        <mesh filename="package://usv16/meshes/back_arm.STL" />
-      </geometry>
-    </collision>
   </link>
-  <joint
-    name="back_arm_link"
-    type="fixed">
+  <joint name="back_arm_link" type="fixed">
     <origin xyz="0.461035796545679 -1.62938510772266 1.80487186338744" rpy="1.70680851480681 0 0" />
     <parent link="Ship" />
@@ -168,15 +82,4 @@
   </joint>
   <link name="platform">
-    <inertial>
-      <origin xyz="1.015 0.038366 -0.508" rpy="0 0 0" />
-      <mass value="33.428" />
-      <inertia
-        ixx="0.0027338"
-        ixy="-0.020382"
-        ixz="1.4515E-09"
-        iyy="0.15196"
-        iyz="1.9469E-10"
-        izz="0.15469" />
-    </inertial>
     <visual>
       <origin xyz="0 0 0" rpy="0 0 0" />
@@ -188,10 +91,4 @@
       </material>
     </visual>
-    <collision>
-      <origin xyz="0 0 0" rpy="0 0 0" />
-      <geometry>
-        <mesh filename="package://usv16/meshes/platform.STL" />
-      </geometry>
-    </collision>
   </link>
   <joint name="platform_link" type="fixed">
@@ -202,15 +99,4 @@
   </joint>
   <link name="owls_nest">
-    <inertial>
-      <origin xyz="7.7996E-05 0.24022 0.074068" rpy="0 0 0" />
-      <mass value="3.138" />
-      <inertia
-        ixx="0.076997"
-        ixy="7.1068E-06"
-        ixz="-7.0107E-05"
-        iyy="0.10637"
-        iyz="0.014352"
-        izz="0.069683" />
-    </inertial>
     <visual>
       <origin xyz="0 0 0" rpy="0 0 0" />
@@ -222,10 +108,4 @@
       </material>
     </visual>
-    <collision>
-      <origin xyz="0 0 0" rpy="0 0 0" />
-      <geometry>
-        <mesh filename="package://usv16/meshes/owls_nest.STL" />
-      </geometry>
-    </collision>
   </link>
   <joint name="owls_nest_link" type="fixed">
@@ -237,5 +117,5 @@
  <xacro:include filename="$(find usv16)/urdf/VLP-16.urdf.xacro"/>
  <VLP-16 parent="platform" name="velodyne" topic="/velodyne_points" hz="10" samples="440">
-   <origin xyz=".2 0.08 -0.5" rpy="1.5707 0 3.14159" />
+   <origin xyz="0 0 0" rpy="1.5707 0 3.14159" />
  </VLP-16>
 </robot>
