Commit message: working lidar simulation but bad coordinates

File: usv16_simulator/urdf/ship.urdf.xacro (robot description, xacro)
@@ -1,4 +1,4 @@
 <?xml version="1.0"?>
-<robot name="Ship">
+<robot xmlns:xacro="http://www.ros.org/wiki/xacro" name="Ship">
   <link name="Ship">
     <visual>
@@ -132,3 +132,7 @@
    <origin xyz="0 0 0"/>
  </joint>
+ <xacro:include filename="$(find usv16)/urdf/VLP-16.urdf.xacro"/>
+ <VLP-16 parent="platform" name="velodyne" topic="/velodyne_points" hz="10" samples="440">
+   <origin xyz="0 0 -1.55" rpy="0 3.14159 3.14159" />
+ </VLP-16>
 </robot>

Commit message: Updates orientation of USV16 model

File: usv16_simulator/urdf/ship.urdf.xacro (robot description, xacro)
@@ -1,237 +1,361 @@
 <?xml version="1.0"?>
 <robot xmlns:xacro="http://www.ros.org/wiki/xacro" name="Ship">
-  <link name="Ship">
-    <inertial>
-      <origin xyz="1.51206787019308 1.78454626473221 0.280594889113911" rpy="0 0 0" />
-      <mass value="0.343059128131347" />
-      <inertia
-        ixx="1.02541857941861E-31"
-        ixy="-1.23259516440783E-32"
-        ixz="-1.7250223049292E-16"
+    <link
+    name="Ship">
+    <inertial>
+      <origin
+        xyz="-0.475299786216409 -0.216942252689994 -0.973841232272509"
+        rpy="0 0 0" />
+      <mass
+        value="0.343059128131347" />
+      <inertia
+        ixx="0.347516126809007"
+        ixy="1.41858996251533E-28"
+        ixz="-1.34839243501966E-14"
         iyy="0.347516126809007"
-        iyz="3.01060216944785E-47"
-        izz="0.347516126809007" />
-    </inertial>
-    <visual>
-      <origin xyz="0 0 0" rpy="0 0 0" />
-      <geometry>
-        <mesh filename="package://usv16/meshes/Ship.STL" />
-      </geometry>
-      <material name="">
-        <color rgba="0.250980392156863 0.250980392156863 0.250980392156863 1" />
-      </material>
-    </visual>
-    <collision>
-      <origin xyz="0 0 0" rpy="0 0 0" />
-      <geometry>
-        <mesh filename="package://usv16/meshes/Ship.STL" />
-      </geometry>
-    </collision>
-  </link>
-  <link name="port_pontoon">
-    <inertial>
-      <origin xyz="2.7149E-05 0.025063 0.96995" rpy="0 0 0" />
-      <mass value="862.28" />
-      <inertia
-        ixx="919.07"
-        ixy="9.5403E-05"
-        ixz="-0.018323"
-        iyy="917.35"
-        iyz="-12.94"
-        izz="1.7236" />
-    </inertial>
-    <visual>
-      <origin xyz="0 0 0" rpy="0 0 0" />
-      <geometry>
-        <mesh filename="package://usv16/meshes/port_pontoon.STL" />
-      </geometry>
-      <material name="">
-        <color rgba="0.50196 0.50196 0.50196 1" />
-      </material>
-    </visual>
-    <collision>
-      <origin xyz="0 0 0" rpy="0 0 0" />
-      <geometry>
-        <mesh filename="package://usv16/meshes/port_pontoon.STL" />
-      </geometry>
-    </collision>
-  </link>
-  <joint name="port_pontoon_link" type="fixed">
-    <origin xyz="2.51854287019308 -1.1575284944847 1.50138062170411" rpy="1.5707963267949 0 0" />
-    <parent link="Ship" />
-    <child link="port_pontoon" />
-    <axis xyz="0 0 0" />
-  </joint>
-  <link name="starboard_pontoon">
-    <inertial>
-      <origin xyz="2.7148E-05 0.025067 0.96992" rpy="0 0 0" />
-      <mass value="862.3" />
-      <inertia
-        ixx="919.13"
-        ixy="9.55E-05"
-        ixz="-0.018324"
-        iyy="917.4"
-        iyz="-12.934"
-        izz="1.7242" />
-    </inertial>
-    <visual>
-      <origin xyz="0 0 0" rpy="0 0 0" />
-      <geometry>
-        <mesh filename="package://usv16/meshes/starboard_pontoon.STL" />
-      </geometry>
-      <material name="">
-        <color rgba="0.50196 0.50196 0.50196 1" />
-      </material>
-    </visual>
-    <collision>
-      <origin xyz="0 0 0" rpy="0 0 0" />
-      <geometry>
-        <mesh filename="package://usv16/meshes/starboard_pontoon.STL" />
-      </geometry>
-    </collision>
-  </link>
-  <joint name="starboard_pontoon_link" type="fixed">
-    <origin xyz="0.505592870193075 -1.1575284944847 1.50138062170411" rpy="1.5707963267949 0 0" />
-    <parent link="Ship" />
-    <child link="starboard_pontoon" />
-    <axis xyz="0 0 0" />
-  </joint>
-  <link name="front_arm">
-    <inertial>
-      <origin xyz="1.035 0.1647 -0.056607" rpy="0 0 0" />
-      <mass value="11.056" />
-      <inertia
-        ixx="0.69846"
-        ixy="0.0042605"
-        ixz="-0.0041643"
-        iyy="3.2431"
-        iyz="-0.32611"
-        izz="3.4715" />
-    </inertial>
-    <visual>
-      <origin xyz="0 0 0" rpy="0 0 0" />
-      <geometry>
-        <mesh filename="package://usv16/meshes/front_arm.STL" />
-      </geometry>
-      <material name="">
-        <color rgba="0.25098 0.25098 0.25098 1" />
-      </material>
-    </visual>
-    <collision>
-      <origin xyz="0 0 0" rpy="0 0 0" />
-      <geometry>
-        <mesh filename="package://usv16/meshes/front_arm.STL" />
-      </geometry>
-    </collision>
-  </link>
-  <joint name="front_arm_link" type="fixed">
-    <origin xyz="0.477017870193075 -3.3012884944847 2.04734366138336" rpy="1.5707963267949 0 0" />
-    <parent link="Ship" />
-    <child link="front_arm" />
-    <axis xyz="0 0 0" />
-  </joint>
-  <link name="back_arm">
-    <inertial>
-      <origin xyz="1.0523 0.53236 -0.046184" rpy="0 0 0" />
-      <mass value="13.904" />
-      <inertia
-        ixx="0.082566"
-        ixy="-0.00023707"
-        ixz="-0.0019543"
-        iyy="0.090768"
-        iyz="-0.0085546"
-        izz="0.017971" />
-    </inertial>
-    <visual>
-      <origin xyz="0 0 0" rpy="0 0 0" />
-      <geometry>
-        <mesh filename="package://usv16/meshes/back_arm.STL" />
-      </geometry>
-      <material name="">
-        <color rgba="0.25098 0.25098 0.25098 1" />
-      </material>
-    </visual>
-    <collision>
-      <origin xyz="0 0 0" rpy="0 0 0" />
-      <geometry>
-        <mesh filename="package://usv16/meshes/back_arm.STL" />
-      </geometry>
-    </collision>
-  </link>
-  <joint
-    name="back_arm_link"
-    type="fixed">
-    <origin xyz="0.461035796545679 -1.62938510772266 1.80487186338744" rpy="1.70680851480681 0 0" />
-    <parent link="Ship" />
-    <child link="back_arm" />
-    <axis xyz="0 0 0" />
-  </joint>
-  <link name="platform">
-    <inertial>
-      <origin xyz="1.015 0.038366 -0.508" rpy="0 0 0" />
-      <mass value="33.428" />
-      <inertia
-        ixx="0.0027338"
-        ixy="-0.020382"
-        ixz="1.4515E-09"
-        iyy="0.15196"
-        iyz="1.9469E-10"
-        izz="0.15469" />
-    </inertial>
-    <visual>
-      <origin xyz="0 0 0" rpy="0 0 0" />
-      <geometry>
-        <mesh filename="package://usv16/meshes/platform.STL" />
-      </geometry>
-      <material name="">
-        <color rgba="0.25098 0.25098 0.25098 1" />
-      </material>
-    </visual>
-    <collision>
-      <origin xyz="0 0 0" rpy="0 0 0" />
-      <geometry>
-        <mesh filename="package://usv16/meshes/platform.STL" />
-      </geometry>
-    </collision>
-  </link>
-  <joint name="platform_link" type="fixed">
-    <origin xyz="2.02006787019308 -3.2631884944847 2.55916499474097" rpy="1.5707963267949 6.12303176911189E-17 1.5707963267949" />
-    <parent link="Ship" />
-    <child link="platform" />
-    <axis xyz="0 0 0" />
-  </joint>
-  <link name="owls_nest">
-    <inertial>
-      <origin xyz="7.7996E-05 0.24022 0.074068" rpy="0 0 0" />
-      <mass value="3.138" />
-      <inertia
-        ixx="0.076997"
-        ixy="7.1068E-06"
-        ixz="-7.0107E-05"
-        iyy="0.10637"
-        iyz="0.014352"
-        izz="0.069683" />
-    </inertial>
-    <visual>
-      <origin xyz="0 0 0" rpy="0 0 0" />
-      <geometry>
-        <mesh filename="package://usv16/meshes/owls_nest.STL" />
-      </geometry>
-      <material name="">
-        <color rgba="0.89804 0.91765 0.92941 1" />
-      </material>
-    </visual>
-    <collision>
-      <origin xyz="0 0 0" rpy="0 0 0" />
-      <geometry>
-        <mesh filename="package://usv16/meshes/owls_nest.STL" />
-      </geometry>
-    </collision>
-  </link>
-  <joint name="owls_nest_link" type="fixed">
-    <origin xyz="1.51206787019308 -1.4597884944847 2.64488999474097" rpy="1.5707963267949 0 0" />
-    <parent link="Ship" />
-    <child link="owls_nest" />
-    <axis xyz="0 0 0" />
+        iyz="3.65608894072494E-15"
+        izz="5.61654659198382E-28" />
+    </inertial>
+    <visual>
+      <origin
+        xyz="0 0 0"
+        rpy="0 0 0" />
+      <geometry>
+        <mesh
+          filename="package://usv16/meshes/Ship.STL" />
+      </geometry>
+      <material
+        name="">
+        <color
+          rgba="0.250980392156863 0.250980392156863 0.250980392156863 1" />
+      </material>
+    </visual>
+    <collision>
+      <origin
+        xyz="0 0 0"
+        rpy="0 0 0" />
+      <geometry>
+        <mesh
+          filename="package://usv16/meshes/Ship.STL" />
+      </geometry>
+    </collision>
+  </link>
+  <link
+    name="port_pontoon">
+    <inertial>
+      <origin
+        xyz="2.71530239263976E-05 -0.025026142464991 -0.970242797822692"
+        rpy="0 0 0" />
+      <mass
+        value="862.145825172756" />
+      <inertia
+        ixx="918.613950239956"
+        ixy="-9.45493204103913E-05"
+        ixz="0.0183165425785058"
+        iyy="916.897716883898"
+        iyz="-12.9964386938207"
+        izz="1.71623425162165" />
+    </inertial>
+    <visual>
+      <origin
+        xyz="0 0 0"
+        rpy="0 0 0" />
+      <geometry>
+        <mesh
+          filename="package://usv16/meshes/port_pontoon.STL" />
+      </geometry>
+      <material
+        name="">
+        <color
+          rgba="0.501960784313725 0.501960784313725 0.501960784313725 1" />
+      </material>
+    </visual>
+    <collision>
+      <origin
+        xyz="0 0 0"
+        rpy="0 0 0" />
+      <geometry>
+        <mesh
+          filename="package://usv16/meshes/port_pontoon.STL" />
+      </geometry>
+    </collision>
+  </link>
+  <joint
+    name="port_pontoon_link"
+    type="fixed">
+    <origin
+      xyz="0.401633819154409 -0.0326337677274606 0.0662233903381412"
+      rpy="1.5707963267949 -6.12303176911189E-17 -1.5707963267949" />
+    <parent
+      link="Ship" />
+    <child
+      link="port_pontoon" />
+    <axis
+      xyz="0 0 0" />
+  </joint>
+  <link
+    name="starboard_pontoon">
+    <inertial>
+      <origin
+        xyz="2.71530237863082E-05 -0.0250261424658662 -0.970242797837432"
+        rpy="0 0 0" />
+      <mass
+        value="862.145825176158" />
+      <inertia
+        ixx="918.61395025306"
+        ixy="-9.45493441066956E-05"
+        ixz="0.0183165425118593"
+        iyy="916.897716896837"
+        iyz="-12.9964386963648"
+        izz="1.71623425178676" />
+    </inertial>
+    <visual>
+      <origin
+        xyz="0 0 0"
+        rpy="0 0 0" />
+      <geometry>
+        <mesh
+          filename="package://usv16/meshes/starboard_pontoon.STL" />
+      </geometry>
+      <material
+        name="">
+        <color
+          rgba="0.501960784313725 0.501960784313725 0.501960784313725 1" />
+      </material>
+    </visual>
+    <collision>
+      <origin
+        xyz="0 0 0"
+        rpy="0 0 0" />
+      <geometry>
+        <mesh
+          filename="package://usv16/meshes/starboard_pontoon.STL" />
+      </geometry>
+    </collision>
+  </link>
+  <joint
+    name="starboard_pontoon_link"
+    type="fixed">
+    <origin
+      xyz="0.401633819154331 1.98031623227254 0.0662233903381622"
+      rpy="1.5707963267949 -6.12303176911189E-17 -1.5707963267949" />
+    <parent
+      link="Ship" />
+    <child
+      link="starboard_pontoon" />
+    <axis
+      xyz="0 0 0" />
+  </joint>
+  <link
+    name="front_arm">
+    <inertial>
+      <origin
+        xyz="1.03496383649083 -0.164697402670872 0.0566073624351731"
+        rpy="0 0 0" />
+      <mass
+        value="11.0557255732339" />
+      <inertia
+        ixx="0.698461968063733"
+        ixy="-0.00426048726717138"
+        ixz="0.00416428496924603"
+        iyy="3.24313575117771"
+        iyz="-0.326114386779029"
+        izz="3.47151383469385" />
+    </inertial>
+    <visual>
+      <origin
+        xyz="0 0 0"
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
Commit message: adds hokuyo and non working fancy gazebo

File: usv16_simulator/urdf/ship.urdf.xacro (robot description, xacro)
@@ -1,19 +1,19 @@
 <?xml version="1.0"?>
-<robot xmlns:xacro="http://www.ros.org/wiki/xacro" name="Ship">
+<robot xmlns:xacro="http://www.ros.org/wiki/xacro" name="wamv">
     <link
     name="Ship">
     <inertial>
       <origin
-        xyz="-0.475299786216409 -0.216942252689994 -0.973841232272509"
-        rpy="0 0 0" />
-      <mass
-        value="0.343059128131347" />
-      <inertia
-        ixx="0.347516126809007"
-        ixy="1.41858996251533E-28"
-        ixz="-1.34839243501966E-14"
-        iyy="0.347516126809007"
-        iyz="3.65608894072494E-15"
-        izz="5.61654659198382E-28" />
+        xyz="-1.17919360537082 -9.06148303321118E-15 0.860343730008724"
+        rpy="0 0 0" />
+      <mass
+        value="0.343059128131349" />
+      <inertia
+        ixx="0.347516126809009"
+        ixy="-3.37337695186157E-15"
+        ixz="-8.26085664640087E-29"
+        iyy="2.41148850167688E-28"
+        iyz="-8.51011003765077E-15"
+        izz="0.347516126809009" />
     </inertial>
     <visual>
@@ -45,15 +45,15 @@
     <inertial>
       <origin
-        xyz="2.71530239263976E-05 -0.025026142464991 -0.970242797822692"
-        rpy="0 0 0" />
-      <mass
-        value="862.145825172756" />
-      <inertia
-        ixx="918.613950239956"
-        ixy="-9.45493204103913E-05"
-        ixz="0.0183165425785058"
-        iyy="916.897716883898"
-        iyz="-12.9964386938207"
-        izz="1.71623425162165" />
+        xyz="0.667982797846472 -1.00650215302528 1.11848323057473"
+        rpy="0 0 0" />
+      <mass
+        value="862.145825161632" />
+      <inertia
+        ixx="1.71623425106692"
+        ixy="0.018316543228869"
+        ixz="12.9964386976976"
+        iyy="918.61395026534"
+        iyz="9.45491027828628E-05"
+        izz="916.897716909836" />
     </inertial>
     <visual>
@@ -85,6 +85,6 @@
     type="fixed">
     <origin
-      xyz="0.401633819154409 -0.0326337677274606 0.0662233903381412"
-      rpy="1.5707963267949 -6.12303176911189E-17 -1.5707963267949" />
+      xyz="0 0 0"
+      rpy="0 0 0" />
     <parent
       link="Ship" />
@@ -98,15 +98,15 @@
     <inertial>
       <origin
-        xyz="2.71530237863082E-05 -0.0250261424658662 -0.970242797837432"
-        rpy="0 0 0" />
-      <mass
-        value="862.145825176158" />
-      <inertia
-        ixx="918.61395025306"
-        ixy="-9.45493441066956E-05"
-        ixz="0.0183165425118593"
-        iyy="916.897716896837"
-        iyz="-12.9964386963648"
-        izz="1.71623425178676" />
+        xyz="0.667982797837398 1.00644784697614 1.118483230571"
+        rpy="0 0 0" />
+      <mass
+        value="862.145825176159" />
+      <inertia
+        ixx="1.71623425178722"
+        ixy="0.0183165425566769"
+        ixz="12.9964386963807"
+        iyy="918.613950253061"
+        iyz="9.45493434948458E-05"
+        izz="916.897716896838" />
     </inertial>
     <visual>
@@ -138,6 +138,6 @@
     type="fixed">
     <origin
-      xyz="0.401633819154331 1.98031623227254 0.0662233903381622"
-      rpy="1.5707963267949 -6.12303176911189E-17 -1.5707963267949" />
+      xyz="0 0 0"
+      rpy="0 0 0" />
     <parent
       link="Ship" />
@@ -151,15 +151,15 @@
     <inertial>
       <origin
-        xyz="1.03496383649083 -0.164697402670872 0.0566073624351731"
-        rpy="0 0 0" />
-      <mass
-        value="11.0557255732339" />
-      <inertia
-        ixx="0.698461968063733"
-        ixy="-0.00426048726717138"
-        ixz="0.00416428496924603"
-        iyy="3.24313575117771"
-        iyz="-0.326114386779029"
-        izz="3.47151383469385" />
+        xyz="1.78456755758353 8.60883452266556E-05 0.433239010214825"
+        rpy="0 0 0" />
+      <mass
+        value="11.0653783507108" />
+      <inertia
+        ixx="3.48329675459449"
+        ixy="0.00416397529788845"
+        ixz="0.327721493095144"
+        iyy="0.701729726060603"
+        iyz="0.00426085885690877"
+        izz="3.25432953655983" />
     </inertial>
     <visual>
@@ -191,6 +191,6 @@
     type="fixed">
     <origin
-      xyz="2.54539381915436 2.00889123227263 -0.479739649340979"
-      rpy="1.5707963267949 -6.12303176911189E-17 -1.5707963267949" />
+      xyz="0 0 0"
+      rpy="0 0 0" />
     <parent
       link="Ship" />
@@ -204,15 +204,15 @@
     <inertial>
       <origin
-        xyz="1.05229885742728 -0.532868649966853 0.046250296402698"
-        rpy="0 0 0" />
-      <mass
-        value="13.890682821647" />
-      <inertia
-        ixx="0.0786723542416337"
-        ixy="0.00022817984044904"
-        ixz="0.00195538317035241"
-        iyy="0.0776647043925609"
-        iyz="-0.00905719116212678"
-        izz="0.00110617465921334" />
+        xyz="0.196024057121332 -0.00126533224415047 0.306308764986796"
+        rpy="0 0 0" />
+      <mass
+        value="13.9035526076094" />
+      <inertia
+        ixx="0.0170110170296931"
+        ixy="0.00196861747276408"
+        ixz="-0.00153977989031901"
+        iyy="0.0825656581724545"
+        iyz="3.0112194497348E-05"
+        izz="0.091728399399986" />
     </inertial>
     <visual>
@@ -241,9 +241,9 @@
   </link>
   <joint
-    name="back_arm"
-    type="fixed">
-    <origin
-      xyz="0.8734904323923 2.02487330591996 -0.237267851345147"
-      rpy="1.70680851480686 -6.12303176911189E-17 -1.5707963267949" />
+    name="back_arm_link"
+    type="fixed">
+    <origin
+      xyz="0 0 0"
+      rpy="0 0 0" />
     <parent
       link="Ship" />
@@ -257,15 +257,15 @@
     <inertial>
       <origin
-        xyz="1.01501521620793 0.0383658735761303 -0.508000009453021"
+        xyz="0.788384783792086 9.45304951461926E-09 0.0473591264239022"
         rpy="0 0 0" />
       <mass
         value="33.4284154923077" />
       <inertia
-        ixx="0.00273377542516084"
-        ixy="-0.020381657490392"
-        ixz="1.45151152451054E-09"
-        iyy="0.151955408711457"
-        iyz="1.94690080378164E-10"
-        izz="0.154689184136618" />
+        ixx="0.00273377542516193"
+        ixy="1.45151924850804E-09"
+        ixz="-0.0203816574903959"
+        iyy="0.154689184136618"
+        iyz="1.94691116391814E-10"
+        izz="0.151955408711456" />
     </inertial>
     <visual>
@@ -297,6 +297,6 @@
     type="fixed">
     <origin
-      xyz="2.50729381915444 0.465841232272631 -0.991560982698607"
-      rpy="-1.5707963267949 4.44089209850067E-14 -3.14159265358979" />
+      xyz="0 0 0"
+      rpy="0 0 0" />
     <parent
       link="Ship" />
@@ -310,15 +310,15 @@
     <inertial>
       <origin
-        xyz="7.79960324067686E-05 -0.240224715837682 -0.074068193355304"
-        rpy="0 0 0" />
-      <mass
-        value="3.1380243003152" />
-      <inertia
-        ixx="0.0769970581968376"
-        ixy="-7.10681264503308E-06"
-        ixz="7.01074722678803E-05"
-        iyy="0.10637093901699"
-        iyz="0.014351686885269"
-        izz="0.0696830731541306" />
+        xyz="0.0740681931076682 -7.79969530188682E-05 -0.240224715486504"
+        rpy="0 0 0" />
+      <mass
+        value="3.13802430797467" />
+      <inertia
+        ixx="0.0696830743963967"
+        ixy="7.01071827526787E-05"
+        ixz="-0.0143516867734258"
+        iyy="0.0769970584322021"
+        iyz="7.10722835819185E-06"
+        izz="0.106370940177521" />
     </inertial>
     <visual>
@@ -350,6 +350,6 @@
     type="fixed">
     <origin
-      xyz="0.70389381915443 0.973841232272564 -1.0772859826987"
-      rpy="1.5707963267949 -6.12303176911189E-17 -1.5707963267949" />
+      xyz="0 0 0"
+      rpy="0 0 0" />
     <parent
       link="Ship" />
@@ -359,7 +359,30 @@
       xyz="0 0 0" />
   </joint>
- <xacro:include filename="$(find usv16)/urdf/VLP-16.urdf.xacro"/>
- <VLP-16 parent="platform" name="velodyne" topic="/velodyne_points" hz="5" samples="110">
-   <origin xyz=".2 0.08 -0.5" rpy="1.5707 0 3.14159" />
- </VLP-16>
+ <xacro:include filename="$(find usv16)/urdf/Hokuyo.urdf.xacro"/>
+  <joint name="hokuyo_joint" type="fixed">
+    <axis xyz="0 1 0" />
+    <origin xyz="1.75 0 0" rpy="0 0 0"/>
+    <parent link="platform"/>
+    <child link="hokuyo_link"/>
+  </joint>
+  <!-- Hokuyo Laser -->
+  <link name="hokuyo_link">
+    <collision>
+      <origin xyz="0 0 0" rpy="0 0 0"/>
+      <geometry>
+        <box size="0.1 0.1 0.1"/>
+      </geometry>
+    </collision>
+    <visual>
+      <origin xyz="0 0 0" rpy="0 0 0"/>
+      <geometry>
+        <mesh filename="package://usv16/meshes/hokuyo.dae"/>
+      </geometry>
+    </visual>
+    <inertial>
+      <mass value="1e-5" />
+      <origin xyz="0 0 0" rpy="0 0 0"/>
+      <inertia ixx="1e-6" ixy="0" ixz="0" iyy="1e-6" iyz="0" izz="1e-6" />
+    </inertial>
+  </link>
 </robot>
